Commit message: version2

File: src/rover_description/urdf/aspha18.urdf (robot description, URDF)
Before this commit: robot rover_description, 10 links, 9 joints
Links:
- added link bio_assembly, mass 5; collision mesh filename=package://rover_description/meshes/bio_assembly.STL scale=0.001 0.001 0.001; visual mesh filename=package://rover_description/meshes/bio_assembly.STL scale=0.001 0.001 0.001
- added link camera_mount, mass 5; collision mesh filename=package://rover_description/meshes/camera_mount.STL scale=0.001 0.001 0.001; visual mesh filename=package://rover_description/meshes/camera_mount.STL scale=0.001 0.001 0.001
- added link com_mount, mass 5; collision mesh filename=package://rover_description/meshes/com_mount.STL scale=0.001 0.001 0.001; visual mesh filename=package://rover_description/meshes/com_mount.STL scale=0.001 0.001 0.001
- link base_rotn: geometry collision mesh filename=package://rover_description/meshes/base_rotation.STL scale=0.001 0.001 0.001; visual mesh filename=package://rover_description/meshes/base_rotation.STL scale=0.001 0.001 0.001
Joints:
- removed joint base_rot1
- added joint base_rotation: type continuous, parent base_link, child base_rotn, origin xyz=0 0.19 0.12 rpy=0 0 0, axis 0 0 1, limit effort=0 velocity=0
- added joint bio_assembly_joint: type fixed, parent base_link, child bio_assembly, origin xyz=0 -0.3 0.1 rpy=0 0 0
- added joint camera_mount_joint: type fixed, parent base_link, child camera_mount, origin xyz=-0.2 0.09 0.12 rpy=0 0 0
- added joint com_mount_joint: type fixed, parent base_link, child com_mount, origin xyz=-0.15 -0.255 0.175 rpy=0 0 0
- joint elbow_joint: origin xyz=0 0.45 0.33 rpy=-0.67 0 0 -> xyz=0 0.43 0.345 rpy=-0.67 0 0
- joint shoulder_joint: origin xyz=0 0 0.02 rpy=0 0 0 -> xyz=0 0.009 0.04 rpy=0 0 0
